File: extension.brd (EAGLE design)
At the start: 156 x 120 mm, 223 parts, among them IC1001 AQV252G2S, IC1002 AQV252G2S, IC1003 AQV252G2S, IC1101 UA78L05ACPK, IC1102 ADUM3300ARW, IC1301 UA78L05ACPK, IC1302 LTC485CS8#PBF, IC1303 ADUM3401ARW, IC1701 ADR3425ARJZ, IC1901 UA78L05ACPK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

Commit message: fixed fuse value in schematic
Parts:
- F1001, F1002, F1003: value 630MA_UMT -> 4,00A_UMT
